Commit message: Initial Commit
Migrate container and simulation configs to ROS Jazzy and enable MoveIt Servo with proper joint limits and mappings.

Key changes:
- Docker/Dockerfile: switch base image from osrf/ros:humble-desktop-full to osrf/ros:jazzy-desktop; update installed ROS package names to jazzy variants; adjust user creation to rename the ubuntu user to 'ros'; add pip install flag (--break-system-packages).
- docker-compose.yml: set DISPLAY to host.docker.internal:0.0 to improve GUI display handling.
- simulation/ros2_ws/src/arm_control/src/arm_controller.cpp: update EEF frame to hand_v111 and remap keyboard joint names to URDF joint names (Revolute_1..6) with comments for joint roles.
- simulation/ros2_ws/src/arm_description/launch/.gitkeep: add placeholder to keep launch directory in VCS.
- simulation/ros2_ws/src/arm_description/urdf/arm.urdf: change joint types from continuous to revolute, add limit elements (lower/upper/effort/velocity) for all revolute joints, and remove transmission blocks (simplify model for simulation).
- simulation/ros2_ws/src/moveit_config/config/joint_limits.yaml: enable velocity and acceleration limits for Revolute_1..6 and set reasonable max_velocity (1.0) and max_acceleration (5.0).
- simulation/ros2_ws/src/moveit_config/config/servo_config.yaml: add Servo configuration tuned for the robot (frames, topics, scaling, publish options, and collision/halt settings).
- simulation/ros2_ws/src/moveit_config/launch/servo.launch.py: add a launch file to start moveit_servo with the new servo configuration and moveit robot descriptions.

Why: these changes align the simulation with the ROS Jazzy environment, enable MoveIt Servo, enforce joint limits for safer and more realistic motion, and ensure joint names and frames match across controller, URDF, and MoveIt configuration.

File: simulation/ros2_ws/src/arm_description/urdf/arm.urdf (robot description, URDF)
Before this commit: robot URDF, 7 links, 6 joints
Joints:
- joint Revolute_1: limit (none) -> lower=-3.14159 upper=3.14159 effort=10.0 velocity=1.0; type continuous -> revolute
- joint Revolute_2: limit (none) -> lower=-3.14159 upper=3.14159 effort=10.0 velocity=1.0; type continuous -> revolute
- joint Revolute_3: limit (none) -> lower=-3.14159 upper=3.14159 effort=10.0 velocity=1.0; type continuous -> revolute
- joint Revolute_4: limit (none) -> lower=-3.14159 upper=3.14159 effort=10.0 velocity=1.0; type continuous -> revolute
- joint Revolute_5: limit (none) -> lower=-3.14159 upper=3.14159 effort=10.0 velocity=1.0; type continuous -> revolute
- joint Revolute_6: limit (none) -> lower=-3.14159 upper=3.14159 effort=10.0 velocity=1.0; type continuous -> revolute
